Commit message: Update package stl file resolution

File: src/annin_ar4_description/urdf/ar_macro.xacro (robot description, xacro)
@@ -28,5 +28,5 @@
     <origin xyz="0 0 0" rpy="0 0 -1.5708"/>
     <geometry>
-      <mesh filename="package://annin_ar4_description/meshes/${robot_parameters['mesh_dir']}/Link_Base_Aluminum.STL"/>
+      <mesh filename="file://$(find annin_ar4_description)/meshes/${robot_parameters['mesh_dir']}/Link_Base_Aluminum.STL"/>
     </geometry>
     <material name="base_aluminum_mat">
@@ -45,5 +45,5 @@
     <origin xyz="0 0 0" rpy="0 0 -1.5708"/>
     <geometry>
-      <mesh filename="package://annin_ar4_description/meshes/${robot_parameters['mesh_dir']}/Link_Base_Enclosure.STL"/>
+      <mesh filename="file://$(find annin_ar4_description)/meshes/${robot_parameters['mesh_dir']}/Link_Base_Enclosure.STL"/>
     </geometry>
     <material name="base_enclosure_mat">
@@ -62,5 +62,5 @@
     <origin xyz="0 0 0" rpy="0 0 -1.5708"/>
     <geometry>
-      <mesh filename="package://annin_ar4_description/meshes/${robot_parameters['mesh_dir']}/Link_Base_Motor.STL"/>
+      <mesh filename="file://$(find annin_ar4_description)/meshes/${robot_parameters['mesh_dir']}/Link_Base_Motor.STL"/>
     </geometry>
     <material name="base_motor_mat">
@@ -90,5 +90,5 @@
     <origin xyz="0 0 0" rpy="0 0 0"/>
     <geometry>
-      <mesh filename="package://annin_ar4_description/meshes/${robot_parameters['mesh_dir']}/Link_1_Aluminum.STL"/>
+      <mesh filename="file://$(find annin_ar4_description)/meshes/${robot_parameters['mesh_dir']}/Link_1_Aluminum.STL"/>
     </geometry>
     <material name="link1_aluminum_mat">
@@ -99,5 +99,5 @@
     <origin xyz="0 0 0" rpy="0 0 0"/>
     <geometry>
-      <mesh filename="package://annin_ar4_description/meshes/${robot_parameters['mesh_dir']}/Link_1_Col.STL"/>
+      <mesh filename="file://$(find annin_ar4_description)/meshes/${robot_parameters['mesh_dir']}/Link_1_Col.STL"/>
     </geometry>
   </collision>
@@ -113,5 +113,5 @@
     <origin xyz="0 0 0" rpy="0 0 0"/>
     <geometry>
-      <mesh filename="package://annin_ar4_description/meshes/${robot_parameters['mesh_dir']}/Link_1_Motor.STL"/>
+      <mesh filename="file://$(find annin_ar4_description)/meshes/${robot_parameters['mesh_dir']}/Link_1_Motor.STL"/>
     </geometry>
     <material name="link1_motors_mat">
@@ -153,5 +153,5 @@
     <origin xyz="0 0 -0.00887" rpy="3.14 0 0"/>
     <geometry>
-      <mesh filename="package://annin_ar4_description/meshes/${robot_parameters['mesh_dir']}/Link_2_Aluminum.STL"/>
+      <mesh filename="file://$(find annin_ar4_description)/meshes/${robot_parameters['mesh_dir']}/Link_2_Aluminum.STL"/>
     </geometry>
     <material name="link2_aluminum_mat">
@@ -162,5 +162,5 @@
     <origin xyz="0 0 -0.00887" rpy="3.14 0 0"/>
     <geometry>
-      <mesh filename="package://annin_ar4_description/meshes/${robot_parameters['mesh_dir']}/Link_2_Col.STL"/>
+      <mesh filename="file://$(find annin_ar4_description)/meshes/${robot_parameters['mesh_dir']}/Link_2_Col.STL"/>
     </geometry>
   </collision>
@@ -177,5 +177,5 @@
     <origin xyz="0 0 -0.00887" rpy="3.14 0 0"/>
     <geometry>
-      <mesh filename="package://annin_ar4_description/meshes/${robot_parameters['mesh_dir']}/Link_2_Motor.STL"/>
+      <mesh filename="file://$(find annin_ar4_description)/meshes/${robot_parameters['mesh_dir']}/Link_2_Motor.STL"/>
     </geometry>
     <material name="link2_motor_mat">
@@ -195,5 +195,5 @@
     <origin xyz="0 0 -0.00887" rpy="3.14 0 0"/>
     <geometry>
-      <mesh filename="package://annin_ar4_description/meshes/${robot_parameters['mesh_dir']}/Link_2_Cover.STL"/>
+      <mesh filename="file://$(find annin_ar4_description)/meshes/${robot_parameters['mesh_dir']}/Link_2_Cover.STL"/>
     </geometry>
     <material name="link2_cover_mat">
@@ -213,5 +213,5 @@
     <origin xyz="0 0 -0.00887" rpy="3.14 0 0"/>
     <geometry>
-      <mesh filename="package://annin_ar4_description/meshes/${robot_parameters['mesh_dir']}/Link_2_Logo.STL"/>
+      <mesh filename="file://$(find annin_ar4_description)/meshes/${robot_parameters['mesh_dir']}/Link_2_Logo.STL"/>
     </geometry>
     <material name="link2_logo_mat">
@@ -253,5 +253,5 @@
     <origin xyz="0 0 -0.03671" rpy="0 0 0"/>
     <geometry>
-      <mesh filename="package://annin_ar4_description/meshes/${robot_parameters['mesh_dir']}/Link_3_Aluminum.STL"/>
+      <mesh filename="file://$(find annin_ar4_description)/meshes/${robot_parameters['mesh_dir']}/Link_3_Aluminum.STL"/>
     </geometry>
     <material name="link3_aluminum_mat">
@@ -262,5 +262,5 @@
     <origin xyz="0 0 -0.03671" rpy="0 0 0"/>
     <geometry>
-      <mesh filename="package://annin_ar4_description/meshes/${robot_parameters['mesh_dir']}/Link_3_Col.STL"/>
+      <mesh filename="file://$(find annin_ar4_description)/meshes/${robot_parameters['mesh_dir']}/Link_3_Col.STL"/>
     </geometry>
   </collision>
@@ -276,5 +276,5 @@
     <origin xyz="0 0 -0.03671" rpy="0 0 0"/>
     <geometry>
-      <mesh filename="package://annin_ar4_description/meshes/${robot_parameters['mesh_dir']}/Link_3_Motor.STL"/>
+      <mesh filename="file://$(find annin_ar4_description)/meshes/${robot_parameters['mesh_dir']}/Link_3_Motor.STL"/>
     </geometry>
     <material name="link3_motor_mat">
@@ -316,5 +316,5 @@
     <origin xyz="0 0 -0.07594" rpy="0 0 -1.5708"/>
     <geometry>
-      <mesh filename="package://annin_ar4_description/meshes/${robot_parameters['mesh_dir']}/Link_4_Aluminum.STL"/>
+      <mesh filename="file://$(find annin_ar4_description)/meshes/${robot_parameters['mesh_dir']}/Link_4_Aluminum.STL"/>
     </geometry>
     <material name="link4_aluminum_mat">
@@ -325,5 +325,5 @@
     <origin xyz="0 0 -0.07594" rpy="0 0 -1.5708"/>
     <geometry>
-      <mesh filename="package://annin_ar4_description/meshes/${robot_parameters['mesh_dir']}/Link_4_Col.STL"/>
+      <mesh filename="file://$(find annin_ar4_description)/meshes/${robot_parameters['mesh_dir']}/Link_4_Col.STL"/>
     </geometry>
   </collision>
@@ -339,5 +339,5 @@
     <origin xyz="0 0 -0.07594" rpy="0 0 -1.5708"/>
     <geometry>
-      <mesh filename="package://annin_ar4_description/meshes/${robot_parameters['mesh_dir']}/Link_4_Motor.STL"/>
+      <mesh filename="file://$(find annin_ar4_description)/meshes/${robot_parameters['mesh_dir']}/Link_4_Motor.STL"/>
     </geometry>
     <material name="link4_motor_mat">
@@ -356,5 +356,5 @@
     <origin xyz="0 0 -0.07594" rpy="0 0 -1.5708"/>
     <geometry>
-      <mesh filename="package://annin_ar4_description/meshes/${robot_parameters['mesh_dir']}/Link_4_Cover.STL"/>
+      <mesh filename="file://$(find annin_ar4_description)/meshes/${robot_parameters['mesh_dir']}/Link_4_Cover.STL"/>
     </geometry>
     <material name="link4_cover_mat">
@@ -373,5 +373,5 @@
     <origin xyz="0 0 -0.07594" rpy="0 0 -1.5708"/>
     <geometry>
-      <mesh filename="package://annin_ar4_description/meshes/${robot_parameters['mesh_dir']}/Link_4_Logo.STL"/>
+      <mesh filename="file://$(find annin_ar4_description)/meshes/${robot_parameters['mesh_dir']}/Link_4_Logo.STL"/>
     </geometry>
     <material name="link4_logo_mat">
@@ -413,5 +413,5 @@
     <origin xyz="0 0 -0.0275" rpy="0 0 0"/>
     <geometry>
-      <mesh filename="package://annin_ar4_description/meshes/${robot_parameters['mesh_dir']}/Link_5_Aluminum.STL"/>
+      <mesh filename="file://$(find annin_ar4_description)/meshes/${robot_parameters['mesh_dir']}/Link_5_Aluminum.STL"/>
     </geometry>
     <material name="aluminum_mat">
@@ -423,5 +423,5 @@
     <origin xyz="0 0 -0.0275" rpy="0 0 0"/>
     <geometry>
-      <mesh filename="package://annin_ar4_description/meshes/${robot_parameters['mesh_dir']}/Link_5_Col.STL"/>
+      <mesh filename="file://$(find annin_ar4_description)/meshes/${robot_parameters['mesh_dir']}/Link_5_Col.STL"/>
     </geometry>
   </collision>
@@ -437,5 +437,5 @@
     <origin xyz="0 0 -0.0275" rpy="0 0 0"/>
     <geometry>
-      <mesh filename="package://annin_ar4_description/meshes/${robot_parameters['mesh_dir']}/Link_5_Motor.STL"/>
+      <mesh filename="file://$(find annin_ar4_description)/meshes/${robot_parameters['mesh_dir']}/Link_5_Motor.STL"/>
     </geometry>
    <material name="motor_mat">
@@ -475,5 +475,5 @@
     <origin xyz="0 0 -0.016" rpy="0 0 0"/>
     <geometry>
-      <mesh filename="package://annin_ar4_description/meshes/${robot_parameters['mesh_dir']}/Link_6_Aluminum.STL"/>
+      <mesh filename="file://$(find annin_ar4_description)/meshes/${robot_parameters['mesh_dir']}/Link_6_Aluminum.STL"/>
     </geometry>
     <material name="aluminum_mat"/>
@@ -483,5 +483,5 @@
     <origin xyz="0 0 -0.016" rpy="0 0 0"/>
     <geometry>
-      <mesh filename="package://annin_ar4_description/meshes/${robot_parameters['mesh_dir']}/Link_6_Col.STL"/>
+      <mesh filename="file://$(find annin_ar4_description)/meshes/${robot_parameters['mesh_dir']}/Link_6_Col.STL"/>
     </geometry>
   </collision>
